File: production/wavewise-ecad/WaveWise_LiftControl/WaveWise_LiftControl.kicad_sch (KiCad schematic)
At the start: 1 part, among them J1 B2B-XH-A

Commit message: rev 1 before merging
lift control rip
Parts:
- removed J1: B2B-XH-A, CONN_B2B-XH-A_JST, symbol 2 pin JST:B2B-XH-A
- added J3: B3B-XH-A, CONN_B3B-XH-A_JST, symbol 3 pin jst:B3B-XH-A
- added J5: B4B-XH-A, CONN_B4B-XH-A_JST, symbol 4 pin jst:B4B-XH-A
- added U1: Raspberry Pi Pico, RPi_Pico:RPi_Pico_SMD_TH, symbol Pico:Pico
- added U1: Pololu_DRV8711_Motor_Driver, Wavewise Footprints UnChecked:POLOLU_36v4, symbol Pololu_Motor_Driver:Pololu_DRV8711_Motor_Driver
Connections:
- new net: J5.4, U1.2 (AOUT1)
- new net: J5.3, U1.3 (AOUT2)
- new net: J5.2, U1.4 (BOUT1)
- new net: J5.1, U1.5 (BOUT2)
- new net +5V: J3.2
- new net +BATT: J3.1, U1.1 (Vin)
- new net GND: J3.3, U1.22 (GND)
- no-connect marks 0 -> 7
Other:
- note added: "Control"
- note added: "Motor Control"
- note added: "Power Input"
