File: production/wavewise-ecad/WaveWise_PMIC/Connectors.kicad_sch (KiCad schematic)
At the start: 9 parts, among them J1 24V output, J10 Signals output, J11 Servo output, J12 Regulated 48V Input, J13 Panel Input, J14 Battery Direct Input, J15 GNDs, J2 12V output, J3 5V output

Commit message: Added Buck converters
Parts:
- removed J1: 24V output, symbol Connector:Screw_Terminal_01x01
- removed J2: 12V output, symbol Connector:Screw_Terminal_01x01
- removed J3: 5V output, symbol Connector:Screw_Terminal_01x01
- added J4: Power outputs, symbol Connector:Screw_Terminal_01x03
Connections:
- net +12V: now also J4.2 (Pin_2)
- net +24V: now also J4.3 (Pin_3)
- net +5V: now also J4.1 (Pin_1)
Other:
- moved on the sheet: J15
