File: production/wavewise-ecad/WaveWise_PMIC/PneumaticControl.kicad_sch (KiCad schematic)
At the start: 8 parts, among them K1 Relay_SPDT, Q2 2N2219, U1 Pololu_DRV8711_Motor_Driver

Commit message: adding more to root page and updating for battery sensing
Parts:
- removed K1: Relay_SPDT, Relay_THT:Relay_SPDT_Finder_36.11, symbol Relay:Relay_SPDT
- added K2: Relay_SPST-NO, symbol Relay:Relay_SPST-NO
- C2: footprint Capacitor_THT:C_Rect_L7.0mm_W2.5mm_P5.00mm -> (none)
- R8: footprint Resistor_SMD:R_0805_2012Metric_Pad1.20x1.40mm_HandSolder -> (none)
Connections:
- net +48V: now also K2.14
- net Inverter_Input: now also K2.13
- net at D2.2 (A), Q2.3 (C): now also K2.A2
- net +5V renamed +12V
- net +12V: now also K2.A1
Changed lines of the file:
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@@
     (effects (font (size 1.27 1.27)) (justify right))
+  )
+  (symbol (lib_id "power:+12V") (at 24.765 43.18 0) (unit 1)
+    (in_bom yes) (on_board yes) (dnp no) (fields_autoplaced)
+    (property "Reference" "#PWR07" (at 24.765 46.99 0)
+      (effects (font (size 1.27 1.27)) hide)
+    )
+    (property "Value" "+12V" (at 24.765 38.1 0)
+      (effects (font (size 1.27 1.27)))
+    )
+    (property "Footprint" "" (at 24.765 43.18 0)
+      (effects (font (size 1.27 1.27)) hide)
+    )
+    (property "Datasheet" "" (at 24.765 43.18 0)
+      (effects (font (size 1.27 1.27)) hide)
+    )
+    (pin "1")
+    (instances
+      (project "WaveWise_PMIC"
+        (path "/8343c01b-8940-4cb8-a17d-91fd7fb1cccd/9401b93a-998f-4185-ba4a-cb0793660d5a"
+          (reference "#PWR07") (unit 1)
+        )
+      )
+    )
   )
   (symbol (lib_id "power:GND") (at 107.696 75.184 0) (unit 1)
@@
         (path "/8343c01b-8940-4cb8-a17d-91fd7fb1cccd/9401b93a-998f-4185-ba4a-cb0793660d5a"
           (reference "#PWR05") (unit 1)
-        )
-      )
-    )
-  )
-  (symbol (lib_id "Relay:Relay_SPDT") (at 40.64 38.1 90) (unit 1)
-    (in_bom yes) (on_board yes) (dnp no) (fields_autoplaced)
-    (property "Reference" "K1" (at 40.64 22.86 90)
-      (effects (font (size 1.27 1.27)))
-    )
-    (property "Value" "Relay_SPDT" (at 40.64 25.4 90)
-      (effects (font (size 1.27 1.27)))
-    )
-    (property "Footprint" "Relay_THT:Relay_SPDT_Finder_36.11" (at 41.91 26.67 0)
-      (effects (font (size 1.27 1.27)) (justify left) hide)
-    )
-    (property "Datasheet" "~" (at 40.64 38.1 0)
-      (effects (font (size 1.27 1.27)) hide)
-    )
-    (pin "11")
-    (pin "A1")
-    (pin "12")
-    (pin "14")
-    (pin "A2")
-    (instances
-      (project "WaveWise_PMIC"
-        (path "/8343c01b-8940-4cb8-a17d-91fd7fb1cccd/9401b93a-998f-4185-ba4a-cb0793660d5a"
-          (reference "K1") (unit 1)
         )
       )
@@
       (effects (font (size 1.27 1.27)) (justify right))
     )
-    (property "Footprint" "Resistor_SMD:R_0805_2012Metric_Pad1.20x1.40mm_HandSolder" (at 57.404 54.356 90)
+    (property "Footprint" "" (at 57.404 54.356 90)
       (effects (font (size 1.27 1.27)) hide)
     )
@@
     )
   )
-  (symbol (lib_id "power:+5V") (at 24.765 43.18 0) (unit 1)
-    (in_bom yes) (on_board yes) (dnp no) (fields_autoplaced)
-    (property "Reference" "#PWR07" (at 24.765 46.99 0)
-      (effects (font (size 1.27 1.27)) hide)
-    )
-    (property "Value" "+5V" (at 24.765 38.1 0)
-      (effects (font (size 1.27 1.27)))
-    )
-    (property "Footprint" "" (at 24.765 43.18 0)
-      (effects (font (size 1.27 1.27)) hide)
-    )
-    (property "Datasheet" "" (at 24.765 43.18 0)
-      (effects (font (size 1.27 1.27)) hide)
-    )
-    (pin "1")
-    (instances
-      (project "WaveWise_PMIC"
-        (path "/8343c01b-8940-4cb8-a17d-91fd7fb1cccd/9401b93a-998f-4185-ba4a-cb0793660d5a"
-          (reference "#PWR07") (unit 1)
+  (symbol (lib_id "Relay:Relay_SPST-NO") (at 40.64 38.1 90) (unit 1)
+    (in_bom yes) (on_board yes) (dnp no)
+    (property "Reference" "K2" (at 47.625 36.83 90)
+      (effects (font (size 1.27 1.27)))
+    )
+    (property "Value" "Relay_SPST-NO" (at 40.64 25.4 90)
+      (effects (font (size 1.27 1.27)))
+    )
+    (property "Footprint" "" (at 41.91 26.67 0)
+      (effects (font (size 1.27 1.27)) (justify left) hide)
+    )
+    (property "Datasheet" "~" (at 40.64 38.1 0)
+      (effects (font (size 1.27 1.27)) hide)
+    )
+    (pin "13")
+    (pin "14")
+    (pin "A1")
+    (pin "A2")
+    (instances
+      (project "WaveWise_PMIC"
+        (path "/8343c01b-8940-4cb8-a17d-91fd7fb1cccd/9401b93a-998f-4185-ba4a-cb0793660d5a"
+          (reference "K2") (unit 1)
         )
       )
@@
       (effects (font (size 1.27 1.27)))
     )
-    (property "Footprint" "Capacitor_THT:C_Rect_L7.0mm_W2.5mm_P5.00mm" (at 32.385 21.9202 0)
-      (effects (font (size 1.27 1.27)) hide)
-    )
+    (property "Footprint" "" (at 32.385 21.9202 0)
+      (effects (font (size 1.27 1.27)) hide)
+    )
