File: production/wavewise-ecad/WaveWise_PMIC/PneumaticControl.kicad_sch (KiCad schematic)
At the start: 6 parts, among them K2 Relay_SPST-NO, Q2 2N2219

Commit message: add control stuff
Parts:
- added R5: 10k, symbol Device:R
- added U1: Pololu_DRV8711_Motor_Driver, Wavewise Footprints UnChecked:POLOLU_36v4, symbol Pololu_Motor_Driver:Pololu_DRV8711_Motor_Driver
Connections:
- net GND: now also R5.2, U1.22 (GND)
- net PUMP_CTRL: now reaches R8.1
- net Inverter_Input: now reaches K2.13, R7.2
- new net +BATT: U1.1 (Vin)
- new net AOUT1: U1.2 (AOUT1)
- new net AOUT2: U1.3 (AOUT2)
- new net BEMF: U1.6 (BEMF)
- new net BOUT1: U1.4 (BOUT1)
- new net BOUT2: U1.5 (BOUT2)
- new net CLK: U1.14 (SCLK)
- new net MISO1: U1.16 (SDATO)
- new net MOSI1: U1.15 (SDATI)
- new net MOTOR_FLT: U1.10 (~FLT)
- new net MOTOR_RESET: R5.1, U1.11 (RST)
- new net SCS: U1.13 (SCS)
- new net STALL: U1.7 (~STALL)
- new net ~SLP: U1.12 (~SLP)
- no-connect marks 0 -> 7
Other:
- note added: "Motor Control"

Commit message: Added some footprints not all yet though
Footprint addition 3/14/2024
Parts:
- C2: value C -> 1uF/100V
- R7: value R_US -> 50; footprint (none) -> Resistor_THT:R_Axial_DIN0516_L15.5mm_D5.0mm_P30.48mm_Horizontal
- R8: value R_US -> 5k
Changed lines of the file:
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@@
       (effects (font (size 1.27 1.27)) (justify right))
     )
-    (property "Value" "R_US" (at 60.325 55.88 0)
+    (property "Value" "5k" (at 60.325 55.88 0)
       (effects (font (size 1.27 1.27)) (justify right))
     )
@@
       (effects (font (size 1.27 1.27)))
     )
-    (property "Value" "R_US" (at 43.815 17.78 90)
+    (property "Value" "50" (at 43.815 17.78 90)
       (effects (font (size 1.27 1.27)))
     )
-    (property "Footprint" "" (at 44.069 19.939 90)
+    (property "Footprint" "Resistor_THT:R_Axial_DIN0516_L15.5mm_D5.0mm_P30.48mm_Horizontal" (at 44.069 19.939 90)
       (effects (font (size 1.27 1.27)) hide)
     )
@@
       (effects (font (size 1.27 1.27)))
     )
-    (property "Value" "C" (at 36.195 16.51 90)
+    (property "Value" "1uF/100V" (at 36.195 16.51 90)
       (effects (font (size 1.27 1.27)))
     )

Commit message: Added more footprints and changed 24V buck shottky diode schematic diagram
Parts:
- removed K2: Relay_SPST-NO, symbol Relay:Relay_SPST-NO
- added K1: Relay_SPDT, Relay_THT:Relay_SPDT_Finder_36.11, symbol Relay:Relay_SPDT
- C2: footprint (none) -> Capacitor_THT:C_Rect_L7.0mm_W2.5mm_P5.00mm
- R8: footprint (none) -> Resistor_SMD:R_0805_2012Metric_Pad1.20x1.40mm_HandSolder
Connections:
- net +48V: now also K1.14
- net Inverter_Input: now also K1.11
- net at D2.2 (A), Q2.3 (C): now also K1.A2
- net +12V renamed +5V
- net +5V: now also K1.A1
Changed lines of the file:
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@@
     (effects (font (size 1.27 1.27)) (justify right))
-  )
-  (symbol (lib_id "power:+12V") (at 24.765 43.18 0) (unit 1)
-    (in_bom yes) (on_board yes) (dnp no) (fields_autoplaced)
-    (property "Reference" "#PWR07" (at 24.765 46.99 0)
-      (effects (font (size 1.27 1.27)) hide)
-    )
-    (property "Value" "+12V" (at 24.765 38.1 0)
-      (effects (font (size 1.27 1.27)))
-    )
-    (property "Footprint" "" (at 24.765 43.18 0)
-      (effects (font (size 1.27 1.27)) hide)
-    )
-    (property "Datasheet" "" (at 24.765 43.18 0)
-      (effects (font (size 1.27 1.27)) hide)
-    )
-    (pin "1")
-    (instances
-      (project "WaveWise_PMIC"
-        (path "/8343c01b-8940-4cb8-a17d-91fd7fb1cccd/9401b93a-998f-4185-ba4a-cb0793660d5a"
-          (reference "#PWR07") (unit 1)
-        )
-      )
-    )
   )
   (symbol (lib_id "power:GND") (at 107.696 75.184 0) (unit 1)
@@
         (path "/8343c01b-8940-4cb8-a17d-91fd7fb1cccd/9401b93a-998f-4185-ba4a-cb0793660d5a"
           (reference "#PWR05") (unit 1)
+        )
+      )
+    )
+  )
+  (symbol (lib_id "Relay:Relay_SPDT") (at 40.64 38.1 90) (unit 1)
+    (in_bom yes) (on_board yes) (dnp no) (fields_autoplaced)
+    (property "Reference" "K1" (at 40.64 22.86 90)
+      (effects (font (size 1.27 1.27)))
+    )
+    (property "Value" "Relay_SPDT" (at 40.64 25.4 90)
+      (effects (font (size 1.27 1.27)))
+    )
+    (property "Footprint" "Relay_THT:Relay_SPDT_Finder_36.11" (at 41.91 26.67 0)
+      (effects (font (size 1.27 1.27)) (justify left) hide)
+    )
+    (property "Datasheet" "~" (at 40.64 38.1 0)
+      (effects (font (size 1.27 1.27)) hide)
+    )
+    (pin "11")
+    (pin "A1")
+    (pin "12")
+    (pin "14")
+    (pin "A2")
+    (instances
+      (project "WaveWise_PMIC"
+        (path "/8343c01b-8940-4cb8-a17d-91fd7fb1cccd/9401b93a-998f-4185-ba4a-cb0793660d5a"
+          (reference "K1") (unit 1)
         )
       )
@@
       (effects (font (size 1.27 1.27)) (justify right))
     )
-    (property "Footprint" "" (at 57.404 54.356 90)
+    (property "Footprint" "Resistor_SMD:R_0805_2012Metric_Pad1.20x1.40mm_HandSolder" (at 57.404 54.356 90)
       (effects (font (size 1.27 1.27)) hide)
     )
@@
     )
   )
-  (symbol (lib_id "Relay:Relay_SPST-NO") (at 40.64 38.1 90) (unit 1)
-    (in_bom yes) (on_board yes) (dnp no)
-    (property "Reference" "K2" (at 47.625 36.83 90)
-      (effects (font (size 1.27 1.27)))
-    )
-    (property "Value" "Relay_SPST-NO" (at 40.64 25.4 90)
-      (effects (font (size 1.27 1.27)))
-    )
-    (property "Footprint" "" (at 41.91 26.67 0)
-      (effects (font (size 1.27 1.27)) (justify left) hide)
-    )
-    (property "Datasheet" "~" (at 40.64 38.1 0)
-      (effects (font (size 1.27 1.27)) hide)
-    )
-    (pin "13")
-    (pin "14")
-    (pin "A1")
-    (pin "A2")
-    (instances
-      (project "WaveWise_PMIC"
-        (path "/8343c01b-8940-4cb8-a17d-91fd7fb1cccd/9401b93a-998f-4185-ba4a-cb0793660d5a"
-          (reference "K2") (unit 1)
+  (symbol (lib_id "power:+5V") (at 24.765 43.18 0) (unit 1)
+    (in_bom yes) (on_board yes) (dnp no) (fields_autoplaced)
+    (property "Reference" "#PWR07" (at 24.765 46.99 0)
+      (effects (font (size 1.27 1.27)) hide)
+    )
+    (property "Value" "+5V" (at 24.765 38.1 0)
+      (effects (font (size 1.27 1.27)))
+    )
+    (property "Footprint" "" (at 24.765 43.18 0)
+      (effects (font (size 1.27 1.27)) hide)
+    )
+    (property "Datasheet" "" (at 24.765 43.18 0)
+      (effects (font (size 1.27 1.27)) hide)
+    )
+    (pin "1")
+    (instances
+      (project "WaveWise_PMIC"
+        (path "/8343c01b-8940-4cb8-a17d-91fd7fb1cccd/9401b93a-998f-4185-ba4a-cb0793660d5a"
+          (reference "#PWR07") (unit 1)
         )
       )
@@
       (effects (font (size 1.27 1.27)))
     )
-    (property "Footprint" "" (at 32.385 21.9202 0)
-      (effects (font (size 1.27 1.27)) hide)
-    )
+    (property "Footprint" "Capacitor_THT:C_Rect_L7.0mm_W2.5mm_P5.00mm" (at 32.385 21.9202 0)
+      (effects (font (size 1.27 1.27)) hide)
+    )

Commit message: Started PCB
Parts:
- Q2: footprint Package_TO_SOT_THT:TO-39-3 -> Package_TO_SOT_THT:TO-92_Inline_Wide
- R5: footprint (none) -> Resistor_SMD:R_0805_2012Metric_Pad1.20x1.40mm_HandSolder
- R7: footprint Resistor_THT:R_Axial_DIN0516_L15.5mm_D5.0mm_P30.48mm_Horizontal -> Resistor_THT:R_Axial_DIN0516_L15.5mm_D5.0mm_P20.32mm_Horizontal
Connections:
- no-connect marks 7 -> 8
Changed lines of the file:
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@@
   (no_connect (at 110.236 59.944))
   (no_connect (at 143.256 33.274))
+  (no_connect (at 33.02 35.56))
   (no_connect (at 143.256 37.084))
   (no_connect (at 110.236 56.134))
@@
       (effects (font (size 1.27 1.27)) (justify left))
     )
-    (property "Footprint" "Package_TO_SOT_THT:TO-39-3" (at 71.12 50.8 0)
+    (property "Footprint" "Package_TO_SOT_THT:TO-92_Inline_Wide" (at 71.12 50.8 0)
       (effects (font (size 1.27 1.27) italic) (justify left) hide)
     )
@@
       (effects (font (size 1.27 1.27)))
     )
-    (property "Footprint" "Resistor_THT:R_Axial_DIN0516_L15.5mm_D5.0mm_P30.48mm_Horizontal" (at 44.069 19.939 90)
+    (property "Footprint" "Resistor_THT:R_Axial_DIN0516_L15.5mm_D5.0mm_P20.32mm_Horizontal" (at 44.069 19.939 90)
       (effects (font (size 1.27 1.27)) hide)
     )
@@
       (effects (font (size 1.27 1.27)) (justify left))
     )
-    (property "Footprint" "" (at 105.918 71.374 90)
-      (effects (font (size 1.27 1.27)) hide)
-    )
+    (property "Footprint" "Resistor_SMD:R_0805_2012Metric_Pad1.20x1.40mm_HandSolder" (at 105.918 71.374 90)
+      (effects (font (size 1.27 1.27)) hide)
+    )
