File: production/wavewise-ecad/WaveWise_PMIC/Power.kicad_sch (KiCad schematic)
At the start: 19 parts, among them IC1 LV14360PDDAR, U1 LM2576HVS-5.0_NOPB

Commit message: Started PCB
Parts:
- removed C1: 100u/80V, Capacitor_THT:CP_Radial_D12.5mm_P5.00mm, symbol Device:C_Polarized_US
- added C1: 100u/80V, Capacitor_THT:CP_Radial_D10.0mm_P5.00mm, symbol Device:C_Polarized
- C6: footprint Wavewise Footprints UnChecked:1000uF_10V_Cap -> Capacitor_THT:CP_Radial_D10.0mm_P5.00mm; symbol Device:C_Polarized_US -> Device:C_Polarized
- R9: footprint (none) -> Resistor_SMD:R_0805_2012Metric_Pad1.20x1.40mm_HandSolder
- renumbered R5 to R14, U1 to U4
Connections:
- net +24V: now also C9.1; no longer C9.P
- net +48V: now also C1.1
- net +5V: now also C6.1; no longer C6.P
- net GND: now also C6.2, C9.2, C1.2; no longer C6.N, C9.N
Changed lines of the file:
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@@
   (symbol (lib_id "Device:R_US") (at 62.23 125.095 0) (unit 1)
     (in_bom yes) (on_board yes) (dnp no) (fields_autoplaced)
-    (property "Reference" "R5" (at 64.77 123.825 0)
+    (property "Reference" "R14" (at 64.77 123.825 0)
       (effects (font (size 1.27 1.27)) (justify left))
     )
@@
       (project "WaveWise_PMIC"
         (path "/8343c01b-8940-4cb8-a17d-91fd7fb1cccd/9b950372-21a2-4bba-abe5-3376787348cc"
-          (reference "R5") (unit 1)
+          (reference "R14") (unit 1)
         )
       )
@@
   (symbol (lib_id "LM2576S-12_NOPB:LM2576S-12_NOPB") (at 126.365 43.18 0) (unit 1)
     (in_bom yes) (on_board yes) (dnp no) (fields_autoplaced)
-    (property "Reference" "U1" (at 126.365 31.75 0)
-      (effects (font (size 1.27 1.27)))
-    )
-    (property "Value" "LM2576HVS-5.0_NOPB" (at 126.365 34.29 0)
+    (property "Reference" "U4" (at 126.365 30.48 0)
+      (effects (font (size 1.27 1.27)))
+    )
+    (property "Value" "LM2576HVS-5.0_NOPB" (at 126.365 33.02 0)
       (effects (font (size 1.27 1.27)))
     )
@@
       (project "WaveWise_PMIC"
         (path "/8343c01b-8940-4cb8-a17d-91fd7fb1cccd/9b950372-21a2-4bba-abe5-3376787348cc"
-          (reference "U1") (unit 1)
+          (reference "U4") (unit 1)
         )
       )
@@
   (symbol (lib_id "power:GND") (at 104.775 50.8 0) (unit 1)
     (in_bom yes) (on_board yes) (dnp no) (fields_autoplaced)
-    (property "Reference" "#PWR017" (at 104.775 57.15 0)
+    (property "Reference" "#PWR0106" (at 104.775 57.15 0)
       (effects (font (size 1.27 1.27)) hide)
     )
@@
       (project "WaveWise_PMIC"
         (path "/8343c01b-8940-4cb8-a17d-91fd7fb1cccd/9b950372-21a2-4bba-abe5-3376787348cc"
-          (reference "#PWR017") (unit 1)
+          (reference "#PWR0106") (unit 1)
         )
       )
@@
   (symbol (lib_id "power:GND") (at 90.805 133.985 0) (unit 1)
     (in_bom yes) (on_board yes) (dnp no) (fields_autoplaced)
-    (property "Reference" "#PWR020" (at 90.805 140.335 0)
+    (property "Reference" "#PWR0101" (at 90.805 140.335 0)
       (effects (font (size 1.27 1.27)) hide)
     )
@@
       (project "WaveWise_PMIC"
         (path "/8343c01b-8940-4cb8-a17d-91fd7fb1cccd/9b950372-21a2-4bba-abe5-3376787348cc"
-          (reference "#PWR020") (unit 1)
+          (reference "#PWR0101") (unit 1)
         )
       )
@@
       (effects (font (size 1.27 1.27)) (justify left))
     )
-    (property "Footprint" "" (at 152.781 127.889 90)
+    (property "Footprint" "Resistor_SMD:R_0805_2012Metric_Pad1.20x1.40mm_HandSolder" (at 152.781 127.889 90)
       (effects (font (size 1.27 1.27)) hide)
     )
@@
     )
   )
-  (symbol (lib_name "C_Polarized_US_1") (lib_id "Device:C_Polarized_US") (at 93.345 46.99 0) (unit 1)
-    (in_bom yes) (on_board yes) (dnp no)
-    (property "Reference" "C1" (at 97.155 48.26 0)
-      (effects (font (size 1.27 1.27)) (justify left))
-    )
-    (property "Value" "100u/80V" (at 93.345 50.8 0)
-      (effects (font (size 1.27 1.27)) (justify left))
-    )
-    (property "Footprint" "Capacitor_THT:CP_Radial_D12.5mm_P5.00mm" (at 93.345 46.99 0)
-      (effects (font (size 1.27 1.27)) hide)
-    )
-    (property "Datasheet" "~" (at 93.345 46.99 0)
-      (effects (font (size 1.27 1.27)) hide)
-    )
-    (pin "N")
-    (pin "P")
-    (instances
-      (project "WaveWise_PMIC"
-        (path "/8343c01b-8940-4cb8-a17d-91fd7fb1cccd/9b950372-21a2-4bba-abe5-3376787348cc"
-          (reference "C1") (unit 1)
-        )
-      )
-    )
-  )
   (symbol (lib_id "power:+48V") (at 52.07 112.395 0) (unit 1)
     (in_bom yes) (on_board yes) (dnp no) (fields_autoplaced)
-    (property "Reference" "#PWR015" (at 52.07 116.205 0)
+    (property "Reference" "#PWR0104" (at 52.07 116.205 0)
       (effects (font (size 1.27 1.27)) hide)
     )
@@
       (project "WaveWise_PMIC"
         (path "/8343c01b-8940-4cb8-a17d-91fd7fb1cccd/9b950372-21a2-4bba-abe5-3376787348cc"
-          (reference "#PWR015") (unit 1)
+          (reference "#PWR0104") (unit 1)
         )
       )
@@
   (symbol (lib_id "power:GND") (at 149.225 50.8 0) (unit 1)
     (in_bom yes) (on_board yes) (dnp no) (fields_autoplaced)
-    (property "Reference" "#PWR031" (at 149.225 57.15 0)
+    (property "Reference" "#PWR0108" (at 149.225 57.15 0)
       (effects (font (size 1.27 1.27)) hide)
     )
@@
       (project "WaveWise_PMIC"
         (path "/8343c01b-8940-4cb8-a17d-91fd7fb1cccd/9b950372-21a2-4bba-abe5-3376787348cc"
-          (reference "#PWR031") (unit 1)
+          (reference "#PWR0108") (unit 1)
         )
       )
@@
   (symbol (lib_id "power:GND") (at 52.07 133.985 0) (unit 1)
     (in_bom yes) (on_board yes) (dnp no) (fields_autoplaced)
-    (property "Reference" "#PWR016" (at 52.07 140.335 0)
+    (property "Reference" "#PWR0103" (at 52.07 140.335 0)
       (effects (font (size 1.27 1.27)) hide)
     )
@@
       (project "WaveWise_PMIC"
         (path "/8343c01b-8940-4cb8-a17d-91fd7fb1cccd/9b950372-21a2-4bba-abe5-3376787348cc"
-          (reference "#PWR016") (unit 1)
+          (reference "#PWR0103") (unit 1)
         )
       )
@@
   (symbol (lib_id "power:GND") (at 93.345 54.61 0) (unit 1)
     (in_bom yes) (on_board yes) (dnp no) (fields_autoplaced)
-    (property "Reference" "#PWR012" (at 93.345 60.96 0)
+    (property "Reference" "#PWR0107" (at 93.345 60.96 0)
       (effects (font (size 1.27 1.27)) hide)
     )
@@
       (project "WaveWise_PMIC"
         (path "/8343c01b-8940-4cb8-a17d-91fd7fb1cccd/9b950372-21a2-4bba-abe5-3376787348cc"
-          (reference "#PWR012") (unit 1)
+          (reference "#PWR0107") (unit 1)
         )
       )
@@
     )
   )
-  (symbol (lib_name "C_Polarized_US_1") (lib_id "Device:C_Polarized_US") (at 165.735 121.92 0) (unit 1)
+  (symbol (lib_id "Device:C_Polarized_US") (at 165.735 121.92 0) (unit 1)
     (in_bom yes) (on_board yes) (dnp no)
     (property "Reference" "C9" (at 169.545 123.19 0)
@@
       (effects (font (size 1.27 1.27)) hide)
     )
-    (pin "N")
-    (pin "P")
+    (pin "2")
+    (pin "1")
     (instances
       (project "WaveWise_PMIC"
@@
   (symbol (lib_id "power:GND") (at 62.23 133.985 0) (unit 1)
     (in_bom yes) (on_board yes) (dnp no) (fields_autoplaced)
-    (property "Reference" "#PWR019" (at 62.23 140.335 0)
+    (property "Reference" "#PWR0102" (at 62.23 140.335 0)
       (effects (font (size 1.27 1.27)) hide)
     )
@@
       (project "WaveWise_PMIC"
         (path "/8343c01b-8940-4cb8-a17d-91fd7fb1cccd/9b950372-21a2-4bba-abe5-3376787348cc"
-          (reference "#PWR019") (unit 1)
+          (reference "#PWR0102") (unit 1)
         )
       )
@@
   (symbol (lib_id "power:+48V") (at 93.345 36.83 0) (unit 1)
     (in_bom yes) (on_board yes) (dnp no) (fields_autoplaced)
-    (property "Reference" "#PWR011" (at 93.345 40.64 0)
+    (property "Reference" "#PWR0105" (at 93.345 40.64 0)
       (effects (font (size 1.27 1.27)) hide)
     )
@@
       (project "WaveWise_PMIC"
         (path "/8343c01b-8940-4cb8-a17d-91fd7fb1cccd/9b950372-21a2-4bba-abe5-3376787348cc"
-          (reference "#PWR011") (unit 1)
+          (reference "#PWR0105") (unit 1)
         )
       )
@@
     )
   )
+  (symbol (lib_id "Device:C_Polarized") (at 93.345 46.99 0) (unit 1)
+    (in_bom yes) (on_board yes) (dnp no) (fields_autoplaced)
+    (property "Reference" "C1" (at 96.52 44.831 0)
+      (effects (font (size 1.27 1.27)) (justify left))
+    )
+    (property "Value" "100u/80V" (at 96.52 47.371 0)
+      (effects (font (size 1.27 1.27)) (justify left))
+    )
+    (property "Footprint" "Capacitor_THT:CP_Radial_D10.0mm_P5.00mm" (at 94.3102 50.8 0)
+      (effects (font (size 1.27 1.27)) hide)
+    )
+    (property "Datasheet" "~" (at 93.345 46.99 0)
+      (effects (font (size 1.27 1.27)) hide)
+    )
+    (pin "1")
+    (pin "2")
+    (instances
+      (project "WaveWise_PMIC"
+        (path "/8343c01b-8940-4cb8-a17d-91fd7fb1cccd/9b950372-21a2-4bba-abe5-3376787348cc"
+          (reference "C1") (unit 1)
+        )
+      )
+    )
+  )
   (symbol (lib_id "Device:R_US") (at 45.72 43.18 0) (unit 1)
     (in_bom yes) (on_board yes) (dnp no) (fields_autoplaced)
@@
     )
   )
-  (symbol (lib_id "Device:C_Polarized_US") (at 169.545 45.72 0) (unit 1)
-    (in_bom yes) (on_board yes) (dnp no) (fields_autoplaced)
-    (property "Reference" "C6" (at 173.355 44.45 0)
-      (effects (font (size 1.27 1.27)) (justify left))
-    )
-    (property "Value" "1000u/10V" (at 173.355 46.99 0)
-      (effects (font (size 1.27 1.27)) (justify left))
-    )
-    (property "Footprint" "Wavewise Footprints UnChecked:1000uF_10V_Cap" (at 169.545 45.72 0)
+  (symbol (lib_id "Device:C_Polarized") (at 169.545 45.72 0) (unit 1)
+    (in_bom yes) (on_board yes) (dnp no) (fields_autoplaced)
+    (property "Reference" "C6" (at 172.72 43.561 0)
+      (effects (font (size 1.27 1.27)) (justify left))
+    )
+    (property "Value" "1000u/10V" (at 172.72 46.101 0)
+      (effects (font (size 1.27 1.27)) (justify left))
+    )
+    (property "Footprint" "Capacitor_THT:CP_Radial_D10.0mm_P5.00mm" (at 170.5102 49.53 0)
       (effects (font (size 1.27 1.27)) hide)
     )
@@
       (effects (font (size 1.27 1.27)) hide)
     )
-    (pin "N")
-    (pin "P")
-    (instances
-      (project "WaveWise_PMIC"
+    (pin "2")
+    (pin "1")
+    (instances
+      (project "WaveWise_PMIC"
