File: production/wavewise-ecad/WaveWise_PMIC/PICO.kicad_sch (KiCad schematic)
At the start: 0 parts

Commit message: Added connectors and pico
Parts:
- added U1: Raspberry Pi Pico, RPi_Pico:RPi_Pico_SMD_TH, symbol Pico:Pico
Changed lines of the file:
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@@
 (kicad_sch (version 20230121) (generator eeschema)
   (paper "A4")
+  (symbol (lib_id "Pico:Pico") (at 56.134 60.198 0) (unit 1)
+    (in_bom yes) (on_board yes) (dnp no) (fields_autoplaced)
+    (property "Reference" "U1" (at 55.499 29.21 0)
+      (effects (font (size 1.27 1.27)))
+    )
+    (property "Value" "Raspberry Pi Pico" (at 55.499 31.75 0)
+      (effects (font (size 1.27 1.27)))
+    )
+    (property "Footprint" "RPi_Pico:RPi_Pico_SMD_TH" (at 57.404 60.198 90)
+      (effects (font (size 1.27 1.27)) hide)
+    )
+    (property "Datasheet" "" (at 57.404 60.198 0)
+      (effects (font (size 1.27 1.27)) hide)
+    )
+    (pin "1")
+    (pin "10")
+    (pin "11")
+    (pin "12")
+    (pin "13")
+    (pin "14")
+    (pin "15")
+    (pin "16")
+    (pin "17")
+    (pin "18")
+    (pin "19")
+    (pin "2")
+    (pin "20")
+    (pin "21")
+    (pin "22")
+    (pin "23")
+    (pin "24")
+    (pin "25")
+    (pin "26")
+    (pin "27")
+    (pin "28")
+    (pin "29")
+    (pin "3")
+    (pin "30")
+    (pin "31")
+    (pin "32")
+    (pin "33")
+    (pin "34")
+    (pin "35")
+    (pin "36")
+    (pin "37")
+    (pin "38")
+    (pin "39")
+    (pin "4")
+    (pin "40")
+    (pin "41")
+    (pin "42")
+    (pin "43")
+    (pin "5")
+    (pin "6")
+    (pin "7")
+    (pin "8")
+    (pin "9")
+    (instances
+      (project "WaveWise_PMIC"
+        (path "/8343c01b-8940-4cb8-a17d-91fd7fb1cccd/448ecc5b-1cdf-4544-9d6c-faff3e79b985"
+          (reference "U1") (unit 1)
+        )
+      )
+    )
+  )
 )

Commit message: add control stuff
Connections:
- net B_TX: now reaches U1.1 (GPIO0)
- net GND: now reaches U1.13 (GND)
- net GND: now also U1.18 (GND), U1.23 (GND), U1.28 (GND), U1.3 (GND), U1.38 (GND), U1.42 (GND), U1.8 (GND)
- net SCK: now reaches U1.14 (GPIO10)
- net MOSI1: now reaches U1.15 (GPIO11)
- net MISO1: now reaches U1.16 (GPIO12)
- net SCS: now reaches U1.17 (GPIO13)
- net ~SLP: now reaches U1.19 (GPIO14)
- net B_RX: now reaches U1.2 (GPIO1)
- net BEMF: now reaches U1.21 (GPIO16)
- net STALL: now reaches U1.22 (GPIO17)
- net GPIO_1: now reaches U1.24 (GPIO18)
- net GPIO_2: now reaches U1.25 (GPIO19)
- net GPIO_3: now reaches U1.26 (GPIO20)
- net GPIO_4: now reaches U1.27 (GPIO21)
- net PUMP_CTRL: now reaches U1.29 (GPIO22)
- net Batt_V_Sense: now reaches U1.31 (GPIO26_ADC0)
- net Panel_V_Sense: now reaches U1.32 (GPIO27_ADC1)
- net +5V: now reaches U1.39 (VSYS)
- net MOTOR_FLT: now reaches U1.4 (GPIO2)
- net CLK: now reaches U1.41 (SWCLK)
- net DIO: now reaches U1.43 (SWDIO)
- net MOTOR_RESET: now reaches U1.5 (GPIO3)
- no-connect marks 0 -> 14
Other:
- moved on the sheet: U1

Commit message: adding more to root page and updating for battery sensing
Connections:
- net Servo: now reaches U1.10 (GPIO7)
- net panelsensDIO: now reaches U1.12 (GPIO9)
- net battsensDIO: now reaches U1.9 (GPIO6)
- net GPIO_4 renamed GPIO4
- no-connect marks 14 -> 11
Changed lines of the file:
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@@
   (paper "A4")
   (no_connect (at 72.898 41.656))
-  (no_connect (at 41.148 44.196))
   (no_connect (at 41.148 39.116))
   (no_connect (at 72.898 36.576))
   (no_connect (at 72.898 31.496))
   (no_connect (at 41.148 72.136))
+  (no_connect (at 72.898 39.116))
   (no_connect (at 41.148 49.276))
-  (no_connect (at 72.898 39.116))
   (no_connect (at 41.148 36.576))
-  (no_connect (at 41.148 46.736))
-  (no_connect (at 41.148 51.816))
   (no_connect (at 72.898 34.036))
   (no_connect (at 72.898 49.276))
@@
     (stroke (width 0) (type default))
   )
+  (wire (pts (xy 40.386 44.196) (xy 41.148 44.196))
+    (stroke (width 0) (type default))
+  )
   (wire (pts (xy 41.148 28.956) (xy 17.526 28.956))
     (stroke (width 0) (type default))
@@
     (stroke (width 0) (type default))
   )
+  (wire (pts (xy 40.386 51.816) (xy 41.148 51.816))
+    (stroke (width 0) (type default))
+  )
   (wire (pts (xy 72.898 26.416) (xy 89.916 26.416))
     (stroke (width 0) (type default))
@@
   )
   (wire (pts (xy 36.322 56.896) (xy 41.148 56.896))
+    (stroke (width 0) (type default))
+  )
+  (wire (pts (xy 40.386 46.736) (xy 41.148 46.736))
     (stroke (width 0) (type default))
   )
@@
     (effects (font (size 1.27 1.27)) (justify left))
   )
+  (hierarchical_label "battsensDIO" (shape input) (at 40.386 44.196 180) (fields_autoplaced)
+    (effects (font (size 1.27 1.27)) (justify right))
+  )
   (hierarchical_label "GPIO_3" (shape input) (at 76.2 59.436 0) (fields_autoplaced)
     (effects (font (size 1.27 1.27)) (justify left))
@@
     (effects (font (size 1.27 1.27)) (justify right))
   )
+  (hierarchical_label "GPIO4" (shape input) (at 76.454 56.896 0) (fields_autoplaced)
+    (effects (font (size 1.27 1.27)) (justify left))
+  )
   (hierarchical_label "Batt_V_Sense" (shape input) (at 76.708 46.736 0) (fields_autoplaced)
     (effects (font (size 1.27 1.27)) (justify left))
   )
+  (hierarchical_label "Servo" (shape input) (at 40.386 46.736 180) (fields_autoplaced)
+    (effects (font (size 1.27 1.27)) (justify right))
+  )
   (hierarchical_label "MISO1" (shape input) (at 36.322 61.976 180) (fields_autoplaced)
+    (effects (font (size 1.27 1.27)) (justify right))
+  )
+  (hierarchical_label "panelsensDIO" (shape input) (at 40.386 51.816 180) (fields_autoplaced)
     (effects (font (size 1.27 1.27)) (justify right))
   )
@@
     (effects (font (size 1.27 1.27)) (justify right))
   )
-  (hierarchical_label "GPIO_4" (shape input) (at 76.454 56.896 0) (fields_autoplaced)
-    (effects (font (size 1.27 1.27)) (justify left))
-  )
   (hierarchical_label "B_RX" (shape input) (at 36.322 26.416 180) (fields_autoplaced)

Commit message: added most footprints still need polulu footprint
Parts:
- U1: footprint RPi_Pico:RPi_Pico_SMD_TH -> Unchecked:Pico
Changed lines of the file:
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@@
       (effects (font (size 1.27 1.27)))
     )
-    (property "Footprint" "RPi_Pico:RPi_Pico_SMD_TH" (at 58.928 48.006 90)
+    (property "Footprint" "Unchecked:Pico" (at 58.928 48.006 90)
       (effects (font (size 1.27 1.27)) hide)
     )

Commit message: Prelim board layout
Connections:
- net panelsensDIO is gone; now on net GPIO4: U1.12 (GPIO9)
- net ~SLP is gone; now on net MOTOR_RESET: U1.19 (GPIO14)
- net Batt_V_Sense: now also U1.32 (GPIO27_ADC1); no longer U1.31 (GPIO26_ADC0)
- net GND: now also U1.33 (AGND)
- net GPIO4: no longer U1.27 (GPIO21)
- net MOTOR_FLT: now also U1.20 (GPIO15); no longer U1.4 (GPIO2)
- net MOTOR_RESET: no longer U1.5 (GPIO3)
- net PUMP_CTRL: now also U1.7 (GPIO5); no longer U1.29 (GPIO22)
- net Panel_V_Sense: now also U1.34 (GPIO28_ADC2); no longer U1.32 (GPIO27_ADC1)
- net Servo: now also U1.6 (GPIO4); no longer U1.10 (GPIO7)
- net GPIO3: now reaches U1.11 (GPIO8)
- net +3.3V: now reaches U1.36 (3V3)
- net BEMF renamed MOTOR_SPI0_RX
- net B_RX renamed UART0_Rx
- net B_TX renamed UART0_TX
- net CLK renamed SWCLK
- net DIO renamed SWDIO
- net GPIO_1 renamed MOTOR_SPI0_SCK
- net GPIO_2 renamed MOTOR_SPI0_TX
- net GPIO_3 renamed MOTOR_DIR/AIN2
- net MISO1: no longer names the net of U1.16 (GPIO12)
- net MOSI1: no longer names the net of U1.15 (GPIO11)
- net SCK: no longer names the net of U1.14 (GPIO10)
- net SCS renamed MOTOR_SLP
- net STALL renamed MOTOR_SPI0_CSn
- net battsensDIO renamed GPIO1
- new net BATT_SENSE_DIO: U1.4 (GPIO2)
- new net GPIO2: U1.10 (GPIO7)
- new net MOTOR_BEMF: U1.31 (GPIO26_ADC0)
- new net MOTOR_STALL: U1.29 (GPIO22)
- new net MOTOR_STEP/AIN1: U1.27 (GPIO21)
- new net PANEL_SENSE_DIO: U1.5 (GPIO3)
- no-connect marks 11 -> 4
Other:
- moved on the sheet: U1

Commit message: power stuff
Connections:
- net PUMP_CTRL renamed BICO_PUMP_CTRL
Changed lines of the file:
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@@
     (effects (font (size 1.27 1.27)) (justify left))
   )
-  (hierarchical_label "PUMP_CTRL" (shape input) (at 35.56 40.64 180) (fields_autoplaced)
+  (hierarchical_label "BICO_PUMP_CTRL" (shape input) (at 35.56 40.64 180) (fields_autoplaced)
     (effects (font (size 1.27 1.27)) (justify right))
   )

Commit message: change pins on pico for layout
Connections:
- net BATT_SENSE_DIO: now also U1.15 (GPIO11); no longer U1.4 (GPIO2)
- net BICO_PUMP_CTRL: now also U1.12 (GPIO9); no longer U1.7 (GPIO5)
- net GPIO1: now also U1.4 (GPIO2); no longer U1.9 (GPIO6)
- net GPIO2: now also U1.5 (GPIO3); no longer U1.10 (GPIO7)
- net GPIO3: now also U1.6 (GPIO4); no longer U1.11 (GPIO8)
- net GPIO4: now also U1.7 (GPIO5); no longer U1.12 (GPIO9)
- net PANEL_SENSE_DIO: now also U1.16 (GPIO12); no longer U1.5 (GPIO3)
- net Servo: now also U1.11 (GPIO8); no longer U1.6 (GPIO4)
Changed lines of the file:
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@@
   (no_connect (at 77.47 50.8))
   (no_connect (at 77.47 25.4))
-  (wire (pts (xy 35.56 38.1) (xy 45.72 38.1))
+  (wire (pts (xy 34.29 50.8) (xy 45.72 50.8))
     (stroke (width 0) (type default))
   )
@@
     (stroke (width 0) (type default))
   )
-  (wire (pts (xy 29.21 50.8) (xy 45.72 50.8))
+  (wire (pts (xy 33.02 38.1) (xy 45.72 38.1))
     (stroke (width 0) (type default))
   )
@@
     (stroke (width 0) (type default))
   )
-  (wire (pts (xy 29.21 45.72) (xy 45.72 45.72))
-    (stroke (width 0) (type default))
-  )
   (wire (pts (xy 77.47 53.34) (xy 81.28 53.34))
     (stroke (width 0) (type default))
   )
-  (wire (pts (xy 35.56 40.64) (xy 45.72 40.64))
+  (wire (pts (xy 33.02 33.02) (xy 45.72 33.02))
     (stroke (width 0) (type default))
   )
@@
     (stroke (width 0) (type default))
   )
+  (wire (pts (xy 34.29 53.34) (xy 45.72 53.34))
+    (stroke (width 0) (type default))
+  )
   (wire (pts (xy 83.82 73.66) (xy 77.47 73.66))
     (stroke (width 0) (type default))
@@
     (stroke (width 0) (type default))
   )
-  (wire (pts (xy 29.21 53.34) (xy 45.72 53.34))
+  (wire (pts (xy 33.02 35.56) (xy 45.72 35.56))
     (stroke (width 0) (type default))
   )
@@
     (stroke (width 0) (type default))
   )
-  (wire (pts (xy 35.56 33.02) (xy 45.72 33.02))
-    (stroke (width 0) (type default))
-  )
   (wire (pts (xy 45.72 68.58) (xy 41.91 68.58))
     (stroke (width 0) (type default))
@@
     (stroke (width 0) (type default))
   )
+  (wire (pts (xy 35.56 60.96) (xy 45.72 60.96))
+    (stroke (width 0) (type default))
+  )
+  (wire (pts (xy 33.02 40.64) (xy 45.72 40.64))
+    (stroke (width 0) (type default))
+  )
   (wire (pts (xy 33.02 27.94) (xy 45.72 27.94))
     (stroke (width 0) (type default))
   )
   (wire (pts (xy 35.56 73.66) (xy 45.72 73.66))
+    (stroke (width 0) (type default))
+  )
+  (wire (pts (xy 35.56 63.5) (xy 45.72 63.5))
     (stroke (width 0) (type default))
   )
@@
     (stroke (width 0) (type default))
   )
-  (wire (pts (xy 35.56 35.56) (xy 45.72 35.56))
-    (stroke (width 0) (type default))
-  )
-  (wire (pts (xy 29.21 48.26) (xy 45.72 48.26))
-    (stroke (width 0) (type default))
-  )
   (wire (pts (xy 33.02 25.4) (xy 45.72 25.4))
     (stroke (width 0) (type default))
@@
     (effects (font (size 1.27 1.27)) (justify left))
   )
-  (hierarchical_label "BATT_SENSE_DIO" (shape input) (at 35.56 33.02 180) (fields_autoplaced)
+  (hierarchical_label "BATT_SENSE_DIO" (shape input) (at 35.56 60.96 180) (fields_autoplaced)
     (effects (font (size 1.27 1.27)) (justify right))
   )
-  (hierarchical_label "GPIO3" (shape input) (at 29.21 50.8 180) (fields_autoplaced)
+  (hierarchical_label "GPIO3" (shape input) (at 33.02 38.1 180) (fields_autoplaced)
     (effects (font (size 1.27 1.27)) (justify right))
   )
-  (hierarchical_label "GPIO1" (shape input) (at 29.21 45.72 180) (fields_autoplaced)
+  (hierarchical_label "GPIO1" (shape input) (at 33.02 33.02 180) (fields_autoplaced)
     (effects (font (size 1.27 1.27)) (justify right))
   )
-  (hierarchical_label "GPIO2" (shape input) (at 29.21 48.26 180) (fields_autoplaced)
+  (hierarchical_label "GPIO2" (shape input) (at 33.02 35.56 180) (fields_autoplaced)
     (effects (font (size 1.27 1.27)) (justify right))
   )
@@
     (effects (font (size 1.27 1.27)) (justify left))
   )
-  (hierarchical_label "GPIO4" (shape input) (at 29.21 53.34 180) (fields_autoplaced)
+  (hierarchical_label "GPIO4" (shape input) (at 33.02 40.64 180) (fields_autoplaced)
     (effects (font (size 1.27 1.27)) (justify right))
   )
@@
     (effects (font (size 1.27 1.27)) (justify left))
   )
-  (hierarchical_label "Servo" (shape input) (at 35.56 38.1 180) (fields_autoplaced)
+  (hierarchical_label "Servo" (shape input) (at 34.29 50.8 180) (fields_autoplaced)
     (effects (font (size 1.27 1.27)) (justify right))
   )
@@
     (effects (font (size 1.27 1.27)) (justify right))
   )
-  (hierarchical_label "PANEL_SENSE_DIO" (shape input) (at 35.56 35.56 180) (fields_autoplaced)
+  (hierarchical_label "PANEL_SENSE_DIO" (shape input) (at 35.56 63.5 180) (fields_autoplaced)
     (effects (font (size 1.27 1.27)) (justify right))
   )
@@
     (effects (font (size 1.27 1.27)) (justify left))
   )
-  (hierarchical_label "BICO_PUMP_CTRL" (shape input) (at 35.56 40.64 180) (fields_autoplaced)
+  (hierarchical_label "BICO_PUMP_CTRL" (shape input) (at 34.29 53.34 180) (fields_autoplaced)
     (effects (font (size 1.27 1.27)) (justify right))
   )
