File: production/wavewise-ecad/WaveWise_Submersible/WaveWise_Submersible.kicad_sch (KiCad schematic)
At the start: 91 parts, among them J1 SMA_CONNECTOR, J10 Screw_Terminal_01x03, J11 Screw_Terminal_01x03, J2 SMA_CONNECTOR, J3 Screw_Terminal_01x04, J4 Screw_Terminal_01x03, J5 SMA_CONNECTOR, J7 Screw_Terminal_01x03, J8 Screw_Terminal_01x03, J8 USB_B_Micro, J9 Screw_Terminal_01x02, M1 MNMOS, M2 MNMOS, U1 ATMEGA328PB-ANR, U2 KP234XTMA1, U3 SI8600AC-B-ISR, U4 EZO_pH_Circuit, U5 SI8600AC-B-ISR, U6 EZO_Conductivity_Circuit, U7 TLV2462CP, U8 FT232RL-REEL, Y1 AS-16.000-20-SMD-TR

Commit message: sub schematic draft
Parts:
- removed C16, C17: 22pF/10V, Capacitor_SMD:C_0805_2012Metric, symbol Device:C
- removed C18, C19, C22, C6, C7, C8: 100n/10V, Capacitor_SMD:C_0805_2012Metric, symbol Device:C
- removed C21: 4.7u/10V, Capacitor_SMD:C_0805_2012Metric, symbol Device:C
- removed D2: 1N5822, Unchecked:1N5822, symbol 1N5822:1N5822
- removed D3, D4: LED_S, LED_THT:LED_D1.8mm_W3.3mm_H2.4mm, symbol Device:LED_Small
- removed J8: USB_B_Micro, WW_Checked:MicroUSB_Mount, symbol Connector:USB_B_Micro
- removed R1, R8: 10k, Resistor_SMD:R_0805_2012Metric, symbol Device:R
- removed R10: 0, Resistor_SMD:R_0805_2012Metric, symbol Device:R
- removed R2, R7, R9: 1k, Resistor_SMD:R_0805_2012Metric, symbol Device:R
- removed R8 (x2): 100, Resistor_SMD:R_0805_2012Metric, symbol Device:R
- removed U1: ATMEGA328PB-ANR, Unchecked:ATMEGA328PB-ANR, symbol ATMEGA328PB-ANR:ATMEGA328PB-ANR
- removed U8: FT232RL-REEL, Unchecked:IC28_SSOP-28_FTD, symbol FT232RL:FT232RL-REEL
- removed UV_INPUT1: TestPoint, TestPoint:TestPoint_Pad_D1.5mm, symbol Connector:TestPoint
- removed Y1: AS-16.000-20-SMD-TR, WW_Checked:WW_Oscillator, symbol Oscillator_16:AS-16.000-20-SMD-TR
- added 12V, 24V, 3V3, VALVE: TestPoint, symbol Connector:TestPoint
- added C11: 22u/10V, Capacitor_SMD:C_0805_2012Metric, symbol Device:C
- added C9: 10u/10V, Capacitor_SMD:C_0805_2012Metric, symbol Device:C
- added J12: Screw_Terminal_01x05, symbol Connector:Screw_Terminal_01x05
- added J14: Screw_Terminal_01x06, symbol Connector:Screw_Terminal_01x06
- added Q1, Q4: Q_NMOS_DGS, symbol Device:Q_NMOS_DGS
- added Q2, Q5: PMOS, symbol Simulation_SPICE:PMOS
- added U10: AZ1117CH-3.3TRG1, Wavewise Footprints UnChecked:SOT-223_DIO, symbol AZ1117CH-3.3TRG1:AZ1117CH-3.3TRG1
- added U9: Raspberry Pi Pico, RPi_Pico:RPi_Pico_SMD_TH, symbol MCU_RaspberryPi_and_Boards:Pico
Connections:
- net +3V3: now also 3V3.1, C11.1, J14.3 (Pin_3), U10.2 (OUTPUT)
- net +5V: now also C9.1, J12.1 (Pin_1), U10.3 (INPUT), U9.39 (VSYS)
- net AIROUT: now also J12.4 (Pin_4), U9.34 (GPIO28_ADC2)
- net EXTGPIO1: now also U9.15 (GPIO11)
- net EXTGPIO2: now also U9.16 (GPIO12)
- net EXTGPIO3: now also U9.17 (GPIO13)
- net EXTGPIO4: now also U9.19 (GPIO14)
- net EXTGPIO5: now also U9.20 (GPIO15)
- net GND1: now also U3.5 (BGND); no longer U3.8 (BGND)
- net GND2: now also U5.5 (BGND); no longer U5.8 (BGND)
- net GNDREF: now also J12.5 (Pin_5), J14.4 (Pin_4), Q1.3 (S), Q4.3 (S), U9.13 (GND), U9.18 (GND), U9.23 (GND), U9.28 (GND), U9.3 (GND), U9.38 (GND), U9.8 (GND)
- net OFF: now also U9.10 (GPIO7)
- net PRESSURE_INPUT: now also U9.32 (GPIO27_ADC1)
- net RESET: now also U9.30 (RUN)
- net SCK0: now also U9.4 (GPIO2)
- net SCL: now also J14.1 (Pin_1), U9.7 (GPIO5)
- net SDA: now also J14.2 (Pin_2), U9.6 (GPIO4)
- net SUB_RX: now also J12.3 (Pin_3), U9.2 (GPIO1)
- net SUB_TX: now also J12.2 (Pin_2), U9.1 (GPIO0)
- net TEMP_INPUT: now also U9.31 (GPIO26_ADC0)
- net VDD: now also U3.8 (BVDD); no longer U3.5 (BVDD)
- net VEE: now also U5.8 (BVDD); no longer U5.5 (BVDD)
- net at R7.2, U4.2 (RX/SCL): now also U3.6 (BSCL); no longer U3.7 (BSCL)
- net at R5.2, U4.3 (TX/SDA): now also U3.7 (BSDA); no longer U3.6 (BSDA)
- net at R12.2, U6.3 (TX/SDA): now also U5.7 (BSDA); no longer U5.6 (BSDA)
- net at R13.2, U6.2 (RX/SCL): now also U5.6 (BSCL); no longer U5.7 (BSCL)
- new net: Q5.2 (G), U9.25 (GPIO19)
- new net: Q1.1 (D), Q2.2 (G), Q4.2 (G), Q5.3 (S)
- new net: Q1.2 (G), U9.24 (GPIO18)
- new net +12V: 12V.1, Q5.1 (D)
- new net +24V: 24V.1, Q2.1 (D)
- new net GND: C11.2, C9.2, U10.1 (ADJ/GND)
- new net READY/INT: J14.5 (Pin_5), U9.9 (GPIO6)
- new net SYNC: J14.6 (Pin_6), U9.11 (GPIO8)
- new net VALVE: Q2.3 (S), Q4.1 (D), VALVE.1
- no-connect marks 31 -> 25
Other:
- note added: "LDO (5V - 3V3)"
- note added: "UV Sensor"
- note removed: "USB Programmer v2"
- moved on the sheet: AIROUT1, GND1, GND2, GNDREF1, OFF1, PRESSURE_INPUT1, RESET1, SCK0, SCL1, SDA1, SUB_RX1, SUB_TX1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

Commit message: Update WaveWise_Submersible.kicad_sch
Changed valve control circuit in sub schematic
Parts:
- removed C13, C15: 0.1uF/10V, Capacitor_SMD:C_0805_2012Metric, symbol Device:C
- removed D1: D_Photo, WW_Checked:GUVA-S12SD, symbol Device:D_Photo
- removed J10, J7: Screw_Terminal_01x03, WW_Checked:ScrewTerminal_01x03_2.54mm, symbol Connector:Screw_Terminal_01x03
- removed J14: Screw_Terminal_01x06, symbol Connector:Screw_Terminal_01x06
- removed R15: 1k, Resistor_SMD:R_0805_2012Metric, symbol Device:R
- removed R19: 1M, Resistor_SMD:R_0805_2012Metric, symbol Device:R
- removed R23: 3.3k, Resistor_SMD:R_0805_2012Metric, symbol Device:R
- removed U7: TLV2462CP, Unchecked:TLV2462CP, symbol TLV2462CP:TLV2462CP
- added J10, J7: Screw_Terminal_01x02, WW_Checked:ScrewTerminal_01x02_2.54mm, symbol Connector:Screw_Terminal_01x02
- added J13: Screw_Terminal_01x04, symbol Connector:Screw_Terminal_01x04
- added J6: Screw_Terminal_01x06, symbol Connector:Screw_Terminal_01x06
- J3: footprint WW_Checked:ScrewTerminal_01x04_2.54mm -> (none)
Connections:
- net +3V3: now also J6.4 (Pin_4)
- net GND: now also U9.42 (GND), J13.2 (Pin_2)
- net GNDREF: now also J10.2 (Pin_2), J6.3 (Pin_3), J7.2 (Pin_2); no longer J3.4 (Pin_4)
- net READY/INT: now also J6.2 (Pin_2)
- net RESET: now also J7.1 (Pin_1)
- net SCK0: now also J3.4 (Pin_4)
- net SCL: now also J6.6 (Pin_6)
- net SDA: now also J6.5 (Pin_5)
- net SYNC: now also J6.1 (Pin_1)
- net VALVE: no longer Q2.3 (S), Q4.1 (D)
- net at Q5.2 (G), U9.25 (GPIO19): now also Q1.2 (G)
- net at U9.24 (GPIO18): no longer Q1.2 (G)
- net SWCLK: now reaches U9.41 (SWCLK)
- net SWCLK: now also J13.1 (Pin_1)
- net SWDIO: now reaches U9.43 (SWDIO)
- net SWDIO: now also J13.3 (Pin_3)
- new net VALVE_IN: J10.1 (Pin_1), Q2.3 (S), Q4.1 (D)
- no-connect marks 25 -> 21
Other:
- note added: "Serial Wire Debug"
- note added: "Valve Control"
- note removed: "UV Sensor + Power Select"
- moved on the sheet: J12, Q1, Q2, Q4, Q5

Commit message: updated mosfet circuit
Parts:
- removed J10, J7, J9: Screw_Terminal_01x02, WW_Checked:ScrewTerminal_01x02_2.54mm, symbol Connector:Screw_Terminal_01x02
- removed J11, J4, J8: Screw_Terminal_01x03, WW_Checked:ScrewTerminal_01x03_2.54mm, symbol Connector:Screw_Terminal_01x03
- removed J12: Screw_Terminal_01x05, symbol Connector:Screw_Terminal_01x05
- removed J13, J3: Screw_Terminal_01x04, symbol Connector:Screw_Terminal_01x04
- removed J6: Screw_Terminal_01x06, symbol Connector:Screw_Terminal_01x06
- removed Q1, Q4: Q_NMOS_DGS, symbol Device:Q_NMOS_DGS
- removed Q2, Q5: PMOS, symbol Simulation_SPICE:PMOS
- added J10, J13: 502584-0270, 5025840270:MOLEX_5025840270, symbol Molex_Clik-Mate:502584-0270
- added J11, J12, J9: 502584-0470, 502584-0470:MOLEX_502584-0470, symbol Molex_Clik-Mate:502584-0470
- added J14, J8: 502584-0370, 502584-0370:MOLEX_502584-0370, symbol Molex_Clik-Mate:502584-0370
- added J4: 502584-0670, 5025840670:MOLEX_5025840670, symbol Molex_Clik-Mate:502584-0670
- added J6: 502584-0570, 5025840570:MOLEX_5025840570, symbol Molex_Clik-Mate:502584-0570
- added U1: IRFL9014TRPBF, SOT-223_VIS, symbol MOSFETs:IRFL9014TRPBF
- added U11: BSS816NWH6327XTSA1, SOT323_BSS816NWH6327XTSA1_INF, symbol MOSFETs:BSS816NWH6327XTSA1
- added U7: NTE4151PT1G, SC89-3_0P95X1P7_ONS, symbol MOSFETs:NTE4151PT1G
- added U8: IRFR7440TRPBF, D-Pak_IRFR7440TRPBF_INF, symbol MOSFETs:IRFR7440TRPBF
Connections:
- net +12V: now also U7.3 (D)
- net +24V: now also U1.1 (D)
- net +3V3: now also J4.4
- net +5V: now also J12.1, J14.1, J6.1, J8.1
- net AIROUT: now also J6.4
- net EXTGPIO1: now also J8.2
- net EXTGPIO2: now also J8.3
- net EXTGPIO3: now also J9.1
- net EXTGPIO4: now also J9.2
- net EXTGPIO5: now also J9.3
- net GND: now also J11.2
- net GNDREF: now also J10.2, J13.2, J14.3, J4.3, J6.5, J9.4, U11.3 (S), U8.3 (S)
- net PRESSURE_INPUT: now also J14.2
- net READY/INT: now also J4.2
- net RESET: now also J10.1
- net SCK0: now also J12.4
- net SCL: now also J4.6
- net SDA: now also J4.5
- net SUB_RX: now also J12.3, J6.3
- net SUB_TX: now also J12.2, J6.2
- net SWCLK: now also J11.1
- net SWDIO: now also J11.3
- net SYNC: now also J4.1
- net VALVE_IN: now also J13.1, U1.3 (S), U8.1 (D)
- net at U9.25 (GPIO19): now also U11.2 (G), U7.1 (G)
- new net: U1.2 (G), U11.1 (D), U7.2 (S), U8.2 (G)
- no-connect marks 21 -> 38

Commit message: changed header pins/valve control
Parts:
- removed J10, J13: 502584-0270, 5025840270:MOLEX_5025840270, symbol Molex_Clik-Mate:502584-0270
- removed J11, J12, J9: 502584-0470, 502584-0470:MOLEX_502584-0470, symbol Molex_Clik-Mate:502584-0470
- removed J8: 502584-0370, 502584-0370:MOLEX_502584-0370, symbol Molex_Clik-Mate:502584-0370
- removed U1: IRFL9014TRPBF, SOT-223_VIS, symbol MOSFETs:IRFL9014TRPBF
- removed U11: BSS816NWH6327XTSA1, SOT323_BSS816NWH6327XTSA1_INF, symbol MOSFETs:BSS816NWH6327XTSA1
- removed U7: NTE4151PT1G, SC89-3_0P95X1P7_ONS, symbol MOSFETs:NTE4151PT1G
- removed U8: IRFR7440TRPBF, D-Pak_IRFR7440TRPBF_INF, symbol MOSFETs:IRFR7440TRPBF
- added C7: C, symbol Device:C
- added D1: 1N5817, Diode_THT:D_DO-41_SOD81_P10.16mm_Horizontal, symbol Diode:1N5817
- added J10: Conn_01x03_Pin, symbol Connector:Conn_01x03_Pin
- added J13: Conn_01x06_Pin, symbol Connector:Conn_01x06_Pin
- added J3, J7: 502584-0270, 5025840270:MOLEX_5025840270, symbol Molex_Clik-Mate:502584-0270
- added J8: Conn_01x07_Pin, symbol Connector:Conn_01x07_Pin
- added K1: Relay_SPST-NO, symbol Relay:Relay_SPST-NO
- added Q1: 2N2219, Package_TO_SOT_THT:TO-39-3, symbol Transistor_BJT:2N2219
- added R15, R16: R_US, symbol Device:R_US
- renumbered AIROUT1 to AIR_INPUT1
Connections:
- net +12V: now also J6.2, D1.1 (K), K1.A1
- net +24V: now also J6.1, C7.2, K1.14
- net +5V: now also J6.3, J13.1 (Pin_1), J8.1 (Pin_1); no longer J6.1
- net EXTGPIO1: now also J8.2 (Pin_2)
- net EXTGPIO2: now also J8.3 (Pin_3)
- net EXTGPIO3: now also J8.4 (Pin_4)
- net EXTGPIO4: now also J8.5 (Pin_5)
- net EXTGPIO5: now also J8.6 (Pin_6)
- net GND: now also J10.2 (Pin_2); no longer C11.2, C9.2, U10.1 (ADJ/GND)
- net GNDREF: now also C11.2, C9.2, U10.1 (ADJ/GND), J13.6 (Pin_6), J3.2, J7.2, J8.7 (Pin_7), Q1.1 (E); no longer J6.5
- net RESET: now also J13.5 (Pin_5)
- net SCK0: now also J13.4 (Pin_4)
- net SUB_RX: now also J6.5, J13.3 (Pin_3); no longer J6.3
- net SUB_TX: now also J6.4, J13.2 (Pin_2); no longer J6.2
- net SWCLK: now also J10.1 (Pin_1)
- net SWDIO: now also J10.3 (Pin_3)
- net VALVE_OUT: now reaches U9.25 (GPIO19)
- net VALVE_OUT: now also R16.1
- net AIROUT renamed AIR_INPUT
- net AIR_INPUT: now also J7.1; no longer J6.4
- new net: J3.1, K1.13, R15.2
- new net: D1.2 (A), K1.A2, Q1.3 (C)
- new net: C7.1, R15.1
- new net: Q1.2 (B), R16.2
- no-connect marks 38 -> 29
Other:
- moved on the sheet: AIR_INPUT1, C11, C9, OFF1, PRESSURE_INPUT1, RESET1, SCK0, SCL1, SDA1, SUB_RX1, SUB_TX1, TEMP_INPUT1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

Commit message: layout first draft, added general/connector footprint
Parts:
- removed 12V: TestPoint, symbol Connector:TestPoint
- removed C5, C6: 1u/10V, Capacitor_SMD:C_0805_2012Metric, symbol Device:C
- removed C7: C, symbol Device:C
- removed D1: 1N5817, Diode_THT:D_DO-41_SOD81_P10.16mm_Horizontal, symbol Diode:1N5817
- removed J14: 502584-0370, 502584-0370:MOLEX_502584-0370, symbol Molex_Clik-Mate:502584-0370
- removed J3, J7: 502584-0270, 5025840270:MOLEX_5025840270, symbol Molex_Clik-Mate:502584-0270
- removed J4: 502584-0670, 5025840670:MOLEX_5025840670, symbol Molex_Clik-Mate:502584-0670
- removed J5: SMA_CONNECTOR, Unchecked:SMA_Jack, symbol SMA_CONNECTOR:SMA_CONNECTOR
- removed J6: 502584-0570, 5025840570:MOLEX_5025840570, symbol Molex_Clik-Mate:502584-0570
- removed K1: Relay_SPST-NO, symbol Relay:Relay_SPST-NO
- removed M1, M2: MNMOS, Unchecked:nMOS_ThroughHole, symbol pspice:MNMOS
- removed OFF1, RESET1, SCK0: TestPoint, TestPoint:TestPoint_Pad_D1.5mm, symbol Connector:TestPoint
- removed Q1: 2N2219, Package_TO_SOT_THT:TO-39-3, symbol Transistor_BJT:2N2219
- removed R10, R11: 1M, Resistor_SMD:R_0805_2012Metric, symbol Device:R
- removed R15, R16: R_US, symbol Device:R_US
- removed R8, R9: 10K, Resistor_SMD:R_0805_2012Metric, symbol Device:R
- added AIR_COMP1, BATT_SENSE1, PANEL_SENSE1: TestPoint, TestPoint:TestPoint_Pad_D1.5mm, symbol Connector:TestPoint
- added C10, C13, C14, C16: 330p, Capacitor_SMD:C_0603_1608Metric, symbol Device:C
- added C12, C15: 6.8u, Capacitor_SMD:C_0603_1608Metric, symbol Device:C
- added C17: 1u, Capacitor_SMD:C_0603_1608Metric, symbol Device:C
- added C8: 0.1u, Capacitor_SMD:C_0603_1608Metric, symbol Device:C
- added D2: 1N5817, Diode_THT:D_DO-41_SOD81_P10.16mm_Horizontal, symbol Diode:1N5817
- added J11: 5031750600, Connector:5031750600, symbol 6pinmolex:5031590600
- added J3: Conn_01x04_Pin, Connector:61300411121, symbol Connector:Conn_01x04_Pin
- added J4: SMA_CONNECTOR, Connector:SMA_Jack, symbol SMA_CONNECTOR:SMA_CONNECTOR
- added J6: 5031750200, Connector:5031750200, symbol 2pinmolex:5031590200
- added J7: 5031750800, Connector:5031750800, symbol 8pinmolex:5031590800
- added J9: 5031750300, Connector:5031750300, symbol 3pinmolex:5031590300
- added K2: AWHSH105D00G, Relay_SMD:AWHSH105D00G, symbol AWHSH105D00G:AWHSH105D00G
- added L1, L2: 22u, Inductor_SMD:L_0603_1608Metric, symbol Device:L
- added Q2: 2N2219, Package_TO_SOT_THT:TO-39-3, symbol Transistor_BJT:2N2219
- added R17: 5k, Resistor_SMD:R_0805_2012Metric, symbol Device:R_US
- added R19, R20, R21: 10k, Resistor_SMD:R_0603_1608Metric, symbol Device:R
- added R22, R23, R24, R25, R26, R27: 0, Resistor_SMD:R_0603_1608Metric, symbol Device:R
- added R9: 50, Resistor_SMD:R_0603_1608Metric, symbol Device:R_US
- added U1: ADS1115IDGSR, Converter_ACDC:SOP50P490X110-10N, symbol Analog:ADS1115IDGSR
- 24V1: renamed from 24V; footprint (none) -> TestPoint:TestPoint_Pad_D1.5mm
- 3V3: footprint (none) -> TestPoint:TestPoint_Pad_D1.5mm
- C1, C4: value 1u/10V -> 1u; footprint Capacitor_SMD:C_0805_2012Metric -> Capacitor_SMD:C_0603_1608Metric; Voltage (none) -> 10V
- C11: value 22u/10V -> 22u; footprint Capacitor_SMD:C_0805_2012Metric -> Capacitor_SMD:C_0603_1608Metric; Voltage (none) -> 10V
- C2, C3: value 100nF/10V -> 100nF; footprint Capacitor_SMD:C_0805_2012Metric -> Capacitor_SMD:C_0603_1608Metric; Voltage (none) -> 10V
- C9: value 10u/10V -> 10u; footprint Capacitor_SMD:C_0805_2012Metric -> Capacitor_SMD:C_0603_1608Metric; Voltage (none) -> 10V
- J1, J2: footprint Unchecked:SMA_Jack -> Connector:SMA_Jack
- J10: footprint (none) -> Connector:61300311121
- J13: footprint (none) -> Connector:61300611121
- J8: footprint (none) -> Connector:61300711121
- PS1, PS2: footprint WW_Checked:RFM-0505S -> Converter_DCDC:RFM-0505S
- R1, R3: value 1M -> 0; footprint Resistor_SMD:R_0805_2012Metric -> Resistor_SMD:R_0603_1608Metric
- R12, R13, R14, R2, R4, R5, R6, R7: footprint Resistor_SMD:R_0805_2012Metric -> Resistor_SMD:R_0603_1608Metric
- U10: footprint Wavewise Footprints UnChecked:SOT-223_DIO -> Package_TO_SOT_SMD:SOT-223_DIO
- U2: footprint Unchecked:XDCR_KP234XTMA1 -> Sensor_Pressure:XDCR_KP234XTMA1
- U3, U5: footprint Unchecked:SOIC127P600X175-8N -> Package_SO:SI8600AC-B-ISR
- U4: footprint WW_Checked:EZO_pH_Circuit -> Sensor:EZO_pH_Circuit
- U6: footprint WW_Checked:EZO_Conductivity_Circuit -> Sensor:EZO_Conductivity_Circuit
- U9: footprint RPi_Pico:RPi_Pico_SMD_TH -> MCU_RaspberryPi_and_Boards:RPi_Pico_SMD_TH
- VALVE1: renamed from VALVE; footprint (none) -> TestPoint:TestPoint_Pad_D1.5mm
- renumbered AIR_INPUT1 to AIR_IN1, PRESSURE_INPUT1 to PRESSURE1, TEMP_INPUT1 to TEMP1
Connections:
- net VALVE is gone; now on net VALVE_OUT: VALVE1.1
- net +24V: now also C17.2, J7.1, K2.3
- net +3V3: now also C8.2, J11.4, R19.1, R20.1, R21.1, U1.8 (VDD)
- net +5V: now also C12.1, C15.1, D2.1 (K), J7.2, J9.1, K2.5, L1.1, L2.1; no longer C1.1, PS1.2 (+VIN), PS2.2 (+VIN), R1.1, R3.1
- net AIR_INPUT: now also U9.32 (GPIO27_ADC1); no longer U9.34 (GPIO28_ADC2)
- net EXTGPIO1: now also U9.26 (GPIO20); no longer U9.15 (GPIO11)
- net EXTGPIO2: now also U9.25 (GPIO19); no longer U9.16 (GPIO12)
- net EXTGPIO3: now also U9.24 (GPIO18); no longer U9.17 (GPIO13)
- net EXTGPIO4: now also U9.22 (GPIO17); no longer U9.19 (GPIO14)
- net EXTGPIO5: now also U9.21 (GPIO16); no longer U9.20 (GPIO15)
- net GND1: now also C13.1
- net GND2: now also C1.2, C16.1
- net GNDREF: now also J2.2, J2.3, J2.4, J2.5, PS1.1 (-VIN), PS2.1 (-VIN), U10.4 (EPAD), C12.2, C13.2, C15.2, C16.2, C8.1, J11.3, J6.2, J7.8, J9.3, Q2.1 (E), U1.1 (ADDR), U1.3 (GND); no longer C1.2, J2.G1, J2.G2, J2.G3, J2.G4
- net PRESSURE_INPUT: now also U9.34 (GPIO28_ADC2), J9.2; no longer U9.32 (GPIO27_ADC1)
- net READY/INT: now also U9.15 (GPIO11), J11.2; no longer U9.9 (GPIO6)
- net SCL: now also J13.5 (Pin_5), J11.6, R20.2, R25.1, R27.1, U1.10 (SCL)
- net SDA: now also J13.4 (Pin_4), J11.5, R21.2, R24.1, R26.1, U1.9 (SDA)
- net SUB_RX: now also J7.4
- net SUB_TX: now also J7.3
- net SYNC: now also U9.14 (GPIO10), J11.1; no longer U9.11 (GPIO8)
- net VALVE_OUT: now also U9.29 (GPIO22), R17.1; no longer U9.25 (GPIO19)
- net VDD: now also C10.1
- net VEE: now also C1.1, C14.1
- net at R7.2, U3.6 (BSCL), U4.2 (RX/SCL): now also R27.2
- net at R5.2, U3.7 (BSDA), U4.3 (TX/SDA): now also R24.2
- net at R3.2: now also U9.10 (GPIO7); no longer PS1.1 (-VIN)
- net at R13.2, U5.6 (BSCL), U6.2 (RX/SCL): now also R25.2
- net at R12.2, U5.7 (BSDA), U6.3 (TX/SDA): now also R26.2
- net at U6.4 (PGND): now also J4.2, J4.3, J4.4, J4.5
- net at U6.5 (PRB): now also J4.1
- net OFF: no longer names the net of R1.2
- net OFF: now also U9.11 (GPIO8); no longer U9.10 (GPIO7)
- net RESET: no longer names the net of U9.30 (RUN)
- net RESET: no longer J13.5 (Pin_5)
- net SCK0: no longer names the net of U9.4 (GPIO2)
- net SCK0: no longer J13.4 (Pin_4)
- new net: C10.2, L1.2, PS1.2 (+VIN)
- new net: C14.2, L2.2, PS2.2 (+VIN)
- new net: C17.1, R9.1
- new net: J6.1, K2.1, R9.2
- new net: D2.2 (A), K2.2, Q2.3 (C)
- new net: Q2.2 (B), R17.2
- new net: J1.2, J1.3, J1.4, J1.5, U4.4 (PGND)
- new net ADC0: J3.4 (Pin_4), R22.1, U1.4 (AIN0)
- new net ADC1: J3.3 (Pin_3), R23.1, U1.5 (AIN1)
- new net ADC2: J3.2 (Pin_2), U1.6 (AIN2)
- new net ADC3: J3.1 (Pin_1), U1.7 (AIN3)
- new net ADC_RDY: R19.2, U1.2 (ALERT/RDY), U9.9 (GPIO6)
- new net AIR_COMP: AIR_COMP1.1, J7.5, U9.17 (GPIO13)
- new net BATTERY_SENSE: BATT_SENSE1.1, J7.6, R1.1, R22.2
- new net PANEL_SENSE: J7.7, PANEL_SENSE1.1, R23.2, R3.1
- no-connect marks 29 -> 17
Other:
- note added: "ADC"
- note added: "ADC Connector"
- note added: "Comms Debug"
- note removed: "Backup Programming"
- moved on the sheet: 24V1, 3V3, 5V1, AIR_IN1, C11, C2, C3, C9, GND1, GND2, GNDREF1, H1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

Commit message: Sub layout draft 2 for chiefs
Parts:
- added R10, R11, R15, R8: 0, Resistor_SMD:R_0603_1608Metric, symbol Device:R
- H1, H2, H3, H4: footprint MountingHole:MountingHole_4.3mm_M4 -> MountingHole:MountingHole_3.2mm_M3_ISO7380_Pad; symbol Mechanical:MountingHole -> Mechanical:MountingHole_Pad
Connections:
- net GNDREF: now also R10.1, R11.1, R15.1, R8.1
- new net: H2.1, R10.2
- new net: H1.1, R8.2
- new net: H3.1, R15.2
- new net: H4.1, R11.2

Commit message: Sub pcb draft 3
Parts:
- removed C8: 0.1u, Capacitor_SMD:C_0603_1608Metric, symbol Device:C
- added C5, C6: 0.1u, Capacitor_SMD:C_0805_2012Metric, symbol Device:C
- C1, C10, C11, C12, C13, C14, C15, C16, C17, C2, C3, C4, C9: footprint Capacitor_SMD:C_0603_1608Metric -> Capacitor_SMD:C_0805_2012Metric
- J11: value 5031750600 -> 55935-0610; footprint Connector:5031750600 -> Connector_Molex:Molex_MicroClasp_55935-0610_1x06_P2.00mm_Horizontal
- J6: value 5031750200 -> 55932-0210; footprint Connector:5031750200 -> Connector_Molex:Molex_MicroClasp_55932-0210_1x02_P2.00mm_Vertical
- J7: value 5031750800 -> 55935-0810; footprint Connector:5031750800 -> Connector_Molex:Molex_MicroClasp_55935-0810_1x08_P2.00mm_Horizontal
- J9: value 5031750300 -> 55932-0310; footprint Connector:5031750300 -> Connector_Molex:Molex_MicroClasp_55932-0310_1x03_P2.00mm_Vertical
- L1, L2: footprint Inductor_SMD:L_0603_1608Metric -> Inductor_SMD:SRP6060FA220M
- R1, R10, R11, R12, R13, R14, R15, R19, R2, R20, R21, R22, R23, R24, R25, R26, R27, R3, R4, R5, R6, R7, R8, R9: footprint Resistor_SMD:R_0603_1608Metric -> Resistor_SMD:R_0805_2012Metric
Connections:
- net +3V3: now also C5.2
- net GNDREF: now also C6.1
- new net: C5.1, C6.2
